File: data/rev0.2/_bk/middle_plate_kicad/nnkb.kicad_pcb (KiCad board)
At the start: 2 copper layers, 250.7 x 111.8 mm, 78 parts, among them SW1 SW_PUSH, SW10 SW_PUSH, SW11 SW_PUSH, SW12 SW_PUSH, SW13 SW_PUSH, SW14 SW_PUSH, SW15 SW_PUSH, SW16 SW_PUSH, SW17 SW_PUSH, SW18 SW_PUSH, SW19 SW_PUSH, SW2 SW_PUSH, SW20 SW_PUSH, SW21 SW_PUSH, SW22 SW_PUSH, SW23 SW_PUSH, SW24 SW_PUSH, SW25 SW_PUSH, SW26 SW_PUSH, SW27 SW_PUSH, SW28 SW_PUSH, SW29 SW_PUSH, SW3 SW_PUSH, SW30 SW_PUSH, SW31 SW_PUSH, SW32 SW_PUSH, SW33 SW_PUSH, SW34 SW_PUSH, SW35 SW_PUSH, SW36 SW_PUSH, SW37 RESET_SWITCH, SW4 SW_PUSH, SW5 SW_PUSH, SW6 SW_PUSH, SW7 SW_PUSH, SW8 SW_PUSH, SW9 SW_PUSH, U1 ProMicro

Commit message: horizonプラグインの使い方を追加
Parts:
- removed D1, D10, D11, D12, D13, D14, D15, D16, D17, D18, D19, D2, D20, D21, D22, D23, D24, D25, D26, D27, D28, D29, D3, D30, D31, D32, D33, D34, D35, D36, D4, D5, D6, D7, D8, D9: D, nowt_parts:Diode_SMD
- removed Ref** (x4): Val**, nowt_parts:spacer_m2_2.2mm
- added D37: WS2812B, nowt_parts:LED_WS2812B_PLCC4_5.0x5.0mm_P3.2mm_middle, F.Cu at (99.7, 58.5)
- added D38: WS2812B, nowt_parts:LED_WS2812B_PLCC4_5.0x5.0mm_P3.2mm_middle, F.Cu at (54.0, 57.0)
- added D39: WS2812B, nowt_parts:LED_WS2812B_PLCC4_5.0x5.0mm_P3.2mm_middle, F.Cu at (52.5, 76.9)
- added D40: WS2812B, nowt_parts:LED_WS2812B_PLCC4_5.0x5.0mm_P3.2mm_middle, F.Cu at (93.3, 96.7)
- added D41: WS2812B, nowt_parts:LED_WS2812B_PLCC4_5.0x5.0mm_P3.2mm_middle, F.Cu at (123.1, 113.1)
- added D42: WS2812B, nowt_parts:LED_WS2812B_PLCC4_5.0x5.0mm_P3.2mm_middle, F.Cu at (192.6, 113.1)
- added D43: WS2812B, nowt_parts:LED_WS2812B_PLCC4_5.0x5.0mm_P3.2mm_middle, F.Cu at (222.4, 96.7)
- added D44: WS2812B, nowt_parts:LED_WS2812B_PLCC4_5.0x5.0mm_P3.2mm_middle, F.Cu at (263.2, 76.9)
- added D45: WS2812B, nowt_parts:LED_WS2812B_PLCC4_5.0x5.0mm_P3.2mm_middle, F.Cu at (261.6, 57.0)
- added D46: WS2812B, nowt_parts:LED_WS2812B_PLCC4_5.0x5.0mm_P3.2mm_middle, F.Cu at (215.9, 58.5)
- SW1, SW10, SW11, SW12, SW13, SW14, SW15, SW16, SW17, SW18, SW19, SW2, SW20, SW21, SW22, SW23, SW24, SW25, SW26, SW27, SW28, SW29, SW3, SW30, SW31, SW32, SW33, SW34, SW35, SW36, SW4, SW5, SW6, SW7, SW8, SW9: footprint nowt_parts:SW_Choc -> nowt_parts:CherryMX_Hotswap_middle
- SW37: footprint nowt_parts:ResetSW_1side -> nowt_parts:ResetSW_1side_back_middle
- U1: footprint nowt_parts:ProMicro_v3.5_mods -> nowt_parts:ProMicro_v3.5_mods_middle
- moved SW37 37.2 mm to (144.8, 77.2), turned to 90 degrees
Routing:
- net row2: track 265.7 -> 0.00 mm, vias 3 -> 0
- net row0: track 264.7 -> 0.00 mm
- net row1: track 256.7 -> 0.00 mm
- net row3: track 187.0 -> 0.00 mm, vias 1 -> 0
- net col0: track 164.4 -> 0.00 mm
- net col9: track 163.5 -> 0.00 mm
- net col7: track 158.3 -> 0.00 mm
- net col2: track 154.6 -> 0.00 mm
- net col1: track 136.9 -> 0.00 mm
- net col8: track 136.7 -> 0.00 mm
- net col6: track 134.0 -> 0.00 mm
- net col3: track 120.1 -> 0.00 mm
- net col5: track 113.7 -> 0.00 mm, vias 1 -> 0
- net col4: track 94.9 -> 0.00 mm
- net GND: track 59.8 -> 0.00 mm
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Other:
- board text added: "nowt36 rev1"
- board text removed: "nowt36lp rev0.1"
