File: data/rev0.2/pcb/nowt36lp.kicad_pcb (KiCad board)
At the start: 2 copper layers, 250.7 x 111.8 mm, 78 parts, among them SW1 SW_PUSH, SW10 SW_PUSH, SW11 SW_PUSH, SW12 SW_PUSH, SW13 SW_PUSH, SW14 SW_PUSH, SW15 SW_PUSH, SW16 SW_PUSH, SW17 SW_PUSH, SW18 SW_PUSH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

Commit message: horizonプラグインの使い方を追加
Routing:
- net row2: track 265.7 -> 286.9 mm
- net row3: track 187.0 -> 196.7 mm, vias 1 -> 2
- net reset: track 44.1 -> 36.9 mm
- net GND: track 59.8 -> 57.9 mm
- net col5: track 113.7 -> 115.3 mm
Other:
- board text added: "nowt36lp rev0.2"
- board text removed: "nowt36lp rev0.1"
